Commit message: Rebase from 'release/kinetic/husky_description'

File: urdf/husky.urdf.xacro (robot description, xacro)
@@ -25,7 +25,4 @@
   <xacro:arg name="laser_xyz" default="$(optenv HUSKY_LMS1XX_XYZ 0.2206 0.0 0.00635)" />
   <xacro:arg name="laser_rpy" default="$(optenv HUSKY_LMS1XX_RPY 0.0 0.0 0.0)" />
-  <xacro:arg name="kinect_enabled" default="false" />
-  <xacro:arg name="kinect_xyz" default="$(optenv HUSKY_KINECT_XYZ 0 0 0)" />
-  <xacro:arg name="kinect_rpy" default="$(optenv HUSKY_KINECT_RPY 0 0.18 3.14)" />
   <xacro:arg name="realsense_enabled" default="false" />
   <xacro:arg name="realsense_xyz" default="$(optenv HUSKY_REALSENSE_XYZ 0 0 0)" />
@@ -39,5 +36,4 @@
   <xacro:include filename="$(find husky_description)/urdf/decorations.urdf.xacro" />
   <xacro:include filename="$(find husky_description)/urdf/wheel.urdf.xacro" />
-  <xacro:include filename="$(find husky_description)/urdf/accessories/kinect_camera.urdf.xacro"/>
   <xacro:include filename="$(find husky_description)/urdf/accessories/intel_realsense.urdf.xacro"/>
   <xacro:include filename="$(find husky_description)/urdf/accessories/sick_lms1xx_mount.urdf.xacro"/>
@@ -129,22 +125,11 @@
     </joint>
   </xacro:if>
-  <!-- top sensor arch; include this if we have either the kinect or realsense enabled -->
-  <xacro:property name="topbar_needed_kinect" value="$(arg kinect_enabled)" />
+  <!-- top sensor arch; include this if we have the realsense enabled -->
   <xacro:property name="topbar_needed_realsense" value="$(arg realsense_enabled)" />
   <!-- In melodic we can treat the above as booleans, but in kinetic they're strings, hence this ugliness... -->
-  <xacro:if value="${topbar_needed_kinect.lower() == 'true' or topbar_needed_kinect == '1' or topbar_needed_realsense == 'true' or topbar_needed_realsense == '1'}">
+  <xacro:if value="${topbar_needed_realsense == 'true' or topbar_needed_realsense == '1'}">
     <xacro:sensor_arch prefix="" parent="top_plate_link">
       <origin xyz="-0.35 0 0.51" rpy="0 0 -3.14"/>
     </xacro:sensor_arch>
-  </xacro:if>
-  <!-- add the kinect for xbox 360 to the topbar if needed -->
-  <!-- NOTE: this camera is considered depricated -->
-  <xacro:if value="$(arg kinect_enabled)">
-    <joint name="kinect_frame_joint" type="fixed">
-      <origin xyz="$(arg kinect_xyz)" rpy="$(arg kinect_rpy)" />
-      <parent link="sensor_arch_mount_link"/>
-      <child link="camera_link"/>
-    </joint>
-    <xacro:kinect_camera prefix="camera" robot_namespace="$(arg robot_namespace)"/>
   </xacro:if>
   <!-- add the intel realsense to the topbar if needed -->

Commit message: Rebase from 'release/foxy/husky_description'

File: urdf/husky.urdf.xacro (robot description, xacro)
@@ -14,32 +14,29 @@
       </plugin>
     </gazebo>
-    <gazebo>
-      <plugin name="$(arg prefix)imu_controller" filename="libhector_gazebo_ros_imu.so">
-        <robotNamespace>$(arg robot_namespace)</robotNamespace>
-        <updateRate>50.0</updateRate>
-        <bodyName>$(arg prefix)base_link</bodyName>
-        <topicName>$(arg prefix)imu/data</topicName>
-        <accelDrift>0.005 0.005 0.005</accelDrift>
-        <accelGaussianNoise>0.005 0.005 0.005</accelGaussianNoise>
-        <rateDrift>0.005 0.005 0.005 </rateDrift>
-        <rateGaussianNoise>0.005 0.005 0.005 </rateGaussianNoise>
-        <headingDrift>0.005</headingDrift>
-        <headingGaussianNoise>0.005</headingGaussianNoise>
-      </plugin>
+    <gazebo reference="$(arg prefix)imu_link">
+      <sensor name="$(arg prefix)imu_sensor" type="imu">
+      <plugin filename="libgazebo_ros_imu_sensor.so" name="$(arg prefix)imu_plugin">
+          <ros>
+            <namespace>$(arg prefix)</namespace>
+            <remapping>~/out:=imu/data_raw</remapping>
+          </ros>
+          <initial_orientation_as_reference>false</initial_orientation_as_reference>
+        </plugin>
+        <always_on>true</always_on>
+        <update_rate>100</update_rate>
+        <visualize>true</visualize>
+      </sensor>
     </gazebo>
-    <gazebo>
-      <plugin name="$(arg prefix)gps_controller" filename="libhector_gazebo_ros_gps.so">
-        <robotNamespace>$(arg robot_namespace)</robotNamespace>
-        <updateRate>40</updateRate>
-        <bodyName>$(arg prefix)base_link</bodyName>
-        <frameId>$(arg prefix)base_link</frameId>
-        <topicName>navsat/fix</topicName>
-        <velocityTopicName>$(arg prefix)navsat/vel</velocityTopicName>
-        <referenceLatitude>49.9</referenceLatitude>
-        <referenceLongitude>8.9</referenceLongitude>
-        <referenceHeading>0</referenceHeading>
-        <referenceAltitude>0</referenceAltitude>
-        <drift>0.0001 0.0001 0.0001</drift>
-      </plugin>
+    <gazebo reference="$(arg prefix)gps_link">
+      <sensor name="$(arg prefix)gps_sensor" type="gps">
+      <plugin filename="libgazebo_ros_gps_sensor.so" name="$(arg prefix)gps_plugin">
+          <ros>
+            <namespace>$(arg prefix)</namespace>
+            <remapping>~/out:=gps/data</remapping>
+          </ros>
+        </plugin>
+        <always_on>true</always_on>
+        <update_rate>10</update_rate>
+      </sensor>
     </gazebo>
   </xacro:if>

File: urdf/husky_macro.urdf.xacro (robot description, xacro)
@@ -73,14 +73,20 @@
       <child link="${prefix}inertial_link" />
     </joint>
-    <!-- IMU Link is the standard mounting position for the UM6 IMU.-->
+    <!-- IMU Link-->
     <!-- Can be modified with environment variables in /etc/ros/setup.bash -->
     <link name="${prefix}imu_link"/>
     <joint name="${prefix}imu_joint" type="fixed">
-      <origin xyz="$(optenv HUSKY_IMU_XYZ 0.19 0 0.149)" rpy="$(optenv HUSKY_IMU_RPY 0 -1.5708 3.1416)" />
+      <origin xyz="$(optenv CPR_IMU_XYZ 0 0 0)" rpy="$(optenv CPR_IMU_RPY 0 0 0)" />
       <parent link="${prefix}base_link" />
       <child link="${prefix}imu_link" />
     </joint>
-    <gazebo reference="${prefix}imu_link">
-    </gazebo>
+    <!-- GPS Link-->
+    <!-- Can be modified with environment variables in /etc/ros/setup.bash -->
+    <link name="${prefix}gps_link"/>
+    <joint name="${prefix}gps_joint" type="fixed">
+      <origin xyz="$(optenv CPR_GPS_XYZ 0 0 0)" rpy="$(optenv CPR_GPS_RPY 0 0 0)" />
+      <parent link="${prefix}base_link" />
+      <child link="${prefix}gps_link" />
+    </joint>
     <!-- Husky wheel macros -->
     <xacro:husky_wheel wheel_prefix="${prefix}front_left">
