Commit message: Rebase from 'upstream'

File: husky_description/urdf/husky.urdf.xacro (robot description, xacro)
@@ -237,15 +237,19 @@
   </xacro:if>
   <!-- Intel Realsense Primary and Secondary -->
-  <xacro:if value="${realsense_model == 'd435'}">
-    <xacro:include filename="$(find realsense2_description)/urdf/_d435.urdf.xacro" />
-  </xacro:if>
-  <xacro:if value="${realsense_model == 'd435i'}">
-    <xacro:include filename="$(find realsense2_description)/urdf/_d435i.urdf.xacro" />
-  </xacro:if>
-  <xacro:if value="${realsense_model == 'd415'}">
-    <xacro:include filename="$(find realsense2_description)/urdf/_d415.urdf.xacro" />
-  </xacro:if>
-  <xacro:if value="${realsense_model == 'd455'}">
-    <xacro:include filename="$(find realsense2_description)/urdf/_d435.urdf.xacro" />
+  <xacro:property name="realsense_enabled" value="$(arg realsense_enabled)"/>
+  <xacro:property name="realsense_secondary_enabled" value="$(arg realsense_secondary_enabled)"/>
+  <xacro:if value="${realsense_enabled or realsense_secondary_enabled}">
+      <xacro:if value="${realsense_model == 'd435'}">
+        <xacro:include filename="$(find realsense2_description)/urdf/_d435.urdf.xacro" />
+      </xacro:if>
+      <xacro:if value="${realsense_model == 'd435i'}">
+        <xacro:include filename="$(find realsense2_description)/urdf/_d435i.urdf.xacro" />
+      </xacro:if>
+      <xacro:if value="${realsense_model == 'd415'}">
+        <xacro:include filename="$(find realsense2_description)/urdf/_d415.urdf.xacro" />
+      </xacro:if>
+      <xacro:if value="${realsense_model == 'd455'}">
+        <xacro:include filename="$(find realsense2_description)/urdf/_d435.urdf.xacro" />
+      </xacro:if>
   </xacro:if>
   <xacro:if value="$(arg realsense_enabled)">
