Commit message: Rebase from 'upstream'

File: husky_description/urdf/accessories/intel_realsense.urdf.xacro (robot description, xacro)
@@ -33,5 +33,4 @@
               <width>${width}</width>
               <height>${height}</height>
-              <!-- TODO: check what format the Realsense hardware delivers and set this to match! -->
               <format>RGB8</format>
             </image>

File: husky_description/urdf/husky.urdf.xacro (robot description, xacro)
@@ -1,6 +1,6 @@
 <?xml version="1.0"?>
-<robot xmlns:xacro="http://ros.org/wiki/xacro" name="$(arg name)">
+<robot xmlns:xacro="http://ros.org/wiki/xacro" name="husky">
   <!-- robot name parameter -->
-  <xacro:arg name="name" default="" />
+  <!-- <xacro:arg name="name" default="" /> -->
   <xacro:arg name="prefix" default="" />
   <xacro:arg name="gazebo_controllers" default="$(find husky_control)/config/control.yaml" />

File: husky_description/urdf/husky_macro.urdf.xacro (robot description, xacro)
@@ -1,22 +1,23 @@
 <?xml version="1.0"?>
 <robot xmlns:xacro="http://ros.org/wiki/xacro">
-  <xacro:arg name="laser_enabled" default="false" />
-  <xacro:arg name="laser_xyz" default="$(optenv HUSKY_LMS1XX_XYZ 0.2206 0.0 0.00635)" />
-  <xacro:arg name="laser_rpy" default="$(optenv HUSKY_LMS1XX_RPY 0.0 0.0 0.0)" />
-  <xacro:arg name="realsense_enabled" default="false" />
-  <xacro:arg name="realsense_xyz" default="$(optenv HUSKY_REALSENSE_XYZ 0 0 0)" />
-  <xacro:arg name="realsense_rpy" default="$(optenv HUSKY_REALSENSE_RPY 0 0 0)" />
-  <xacro:arg name="realsense_mount" default="$(optenv HUSKY_REALSENSE_MOUNT_FRAME sensor_arch_mount_link)" />
+  <xacro:arg name="laser_enabled" default="$(optenv CPR_LASER_ENABLED 0)" />
+  <xacro:arg name="laser_xyz" default="$(optenv CPR_LASER_XYZ 0.2206 0.0 0.00635)" />
+  <xacro:arg name="laser_rpy" default="$(optenv CPR_LASER_RPY 0.0 0.0 0.0)" />
+  <xacro:arg name="realsense_enabled" default="$(optenv CPR_REALSENSE 0)" />
+  <xacro:arg name="realsense_xyz" default="$(optenv CPR_REALSENSE_XYZ 0 0 0)" />
+  <xacro:arg name="realsense_rpy" default="$(optenv CPR_REALSENSE_RPY 0 0 0)" />
+  <xacro:arg name="realsense_mount" default="$(optenv CPR_REALSENSE_MOUNT_FRAME sensor_arch_mount_link)" />
   <xacro:property name="husky_front_bumper_extend" value="$(optenv HUSKY_FRONT_BUMPER_EXTEND 0)" />
   <xacro:property name="husky_rear_bumper_extend" value="$(optenv HUSKY_REAR_BUMPER_EXTEND 0)" />
   <xacro:arg name="robot_namespace" default="/" />
   <xacro:arg name="is_sim" default="false" />
-  <xacro:arg name="urdf_extras" default="empty.urdf" />
+  <xacro:arg name="urdf_extras" default="$(optenv CPR_URDF_EXTRAS empty.urdf)" />
+  <xacro:arg name="serial_port" default="$(optenv HUSKY_SERIAL_PORT /dev/prolific)" />
   <!-- Included URDF/XACRO Files -->
   <xacro:include filename="$(find husky_description)/urdf/decorations.urdf.xacro" />
   <xacro:include filename="$(find husky_description)/urdf/wheel.urdf.xacro" />
-  <!-- <xacro:include filename="$(find husky_description)/urdf/accessories/intel_realsense.urdf.xacro"/>
-  <xacro:include filename="$(find husky_description)/urdf/accessories/sick_lms1xx_mount.urdf.xacro"/>
-  <xacro:include filename="$(find husky_description)/urdf/accessories/sensor_arch.urdf.xacro"/> -->
+  <xacro:include filename="$(find husky_description)/urdf/accessories/intel_realsense.urdf.xacro"/>
+  <!-- <xacro:include filename="$(find husky_description)/urdf/accessories/sick_lms1xx_mount.urdf.xacro"/> -->
+  <xacro:include filename="$(find husky_description)/urdf/accessories/sensor_arch.urdf.xacro"/>
   <xacro:property name="M_PI" value="3.14159"/>
   <xacro:macro name="husky" params="prefix">
@@ -37,5 +38,5 @@
         <origin xyz="0 0 0" rpy="0 0 0" />
         <geometry>
-          <mesh filename="file://$(find husky_description)/meshes/base_link.dae" />
+          <mesh filename="package://husky_description/meshes/base_link.dae" />
         </geometry>
       </visual>
@@ -124,13 +125,13 @@
     </xacro:if> -->
     <!-- add the intel realsense to the topbar if needed -->
-    <!-- <xacro:if value="$(arg realsense_enabled)">
+    <xacro:if value="$(arg realsense_enabled)">
       <link name="realsense_mountpoint"/>
       <joint name="realsense_mountpoint_joint" type="fixed">
-        <origin xyz="0 0 0" rpy="0 0 -3.14159" />
+        <origin xyz="$(arg realsense_xyz)" rpy="$(arg realsense_rpy)" />
         <parent link="$(arg realsense_mount)"/>
         <child link="realsense_mountpoint" />
       </joint>
       <xacro:intel_realsense_mount prefix="camera" topic="realsense" parent_link="realsense_mountpoint"/>
-    </xacro:if> -->
+    </xacro:if>
     <ros2_control name="${prefix}husky_hardware" type="system">
       <hardware>
@@ -146,6 +147,6 @@
           <param name="max_accel">5.0</param>
           <param name="max_speed">1.0</param>
-          <param name="polling_timeout">10.0</param>
-          <param name="serial_port">/dev/prolific</param>
+          <param name="polling_timeout">0.1</param>
+          <param name="serial_port">$(arg serial_port)</param>
         </xacro:unless>
       </hardware>
