Commit message: Imported upstream version '0.6.10' of 'upstream'

File: husky_description/urdf/accessories/hokuyo_ust10.urdf.xacro (robot description, xacro)
@@ -62,4 +62,16 @@
         <material name="dark_grey" />
       </visual>
+      <collision>
+        <origin xyz="0 0 0.0175" rpy="0 0 0" />
+        <geometry>
+          <box size="0.05 0.05 0.035" />
+        </geometry>
+      </collision>
+      <collision>
+        <origin xyz="0 0 0.035" rpy="0 0 0" />
+        <geometry>
+          <cylinder radius="0.024" length="0.07" />
+        </geometry>
+      </collision>
     </link>
     <joint name="${prefix}_laser_joint" type="fixed">
